File: hardware_design/V0.2/Hardware/Circuit/main_board_new/Vibration_Sensor/Vibration_Sensor.kicad_pcb (KiCad board)
At the start: 2 copper layers, 65 x 37.6 mm, 13 parts, among them U1 power_input, U2 Teensy4.0-teensy, U5 main_board_top_rail

Commit message: Updated kicad and beam testing files
Parts:
- Teensy 4.0: renamed from U2
- renumbered D1 to LED, Micro_SD1 to Micro_SD, U1 to Power, switch1 to Switch
Connections:
- Teensy 4.0 pad 15: Net-(Micro_SD1-Pad4) -> Net-(U2-Pad15)
- Teensy 4.0 pad 20: Net-(U2-Pad20) -> Net-(Micro_SD1-Pad4)
Routing:
- net Net-(Micro_SD1-Pad4): track 33.2 -> 31.9 mm, vias 0 -> 1
