File: hardware_design/V0.3/Hardware/Circuit/main_board/Vibration_Sensor/Vibration_Sensor.sch (KiCad schematic (older format))
At the start: 16 parts, among them U1 power_input, U2 Teensy4.0-teensy, U3 AP7361C-33E, U4 AP7361C-33E, U5 main_board_top_rail, U6 nRF24L01+, U7 DS3231M

Commit message: PCB changes
Parts:
- Micro_SD1: symbol ARTS-Lab:microSD_small -> Vibration_Sensor-rescue:microSD_small-ARTS-Lab
- U1: symbol ARTS-Lab:power_input -> Vibration_Sensor-rescue:power_input-ARTS-Lab
- U2: symbol ARTS-Lab:Teensy4.0-teensy -> Vibration_Sensor-rescue:Teensy4.0-teensy-ARTS-Lab
- U5: symbol ARTS-Lab:main_board_top_rail -> Vibration_Sensor-rescue:main_board_top_rail-ARTS-Lab
- U6: symbol ARTS-Lab:nRF24L01+ -> Vibration_Sensor-rescue:nRF24L01+-ARTS-Lab
- switch1: symbol ARTS-Lab:grounded_DIP_switch -> Vibration_Sensor-rescue:grounded_DIP_switch-ARTS-Lab
Changed lines of the file:
@@
 $EndDescr
 $Comp
-L ARTS-Lab:Teensy4.0-teensy U2
+L Vibration_Sensor-rescue:Teensy4.0-teensy-ARTS-Lab U2
 U 1 1 6290ED71
 P 3200 3950
@@
 $EndComp
 $Comp
-L ARTS-Lab:microSD_small Micro_SD1
+L Vibration_Sensor-rescue:microSD_small-ARTS-Lab Micro_SD1
 U 1 1 62911122
 P 6900 4350
@@
 $EndComp
 $Comp
-L ARTS-Lab:main_board_top_rail U5
+L Vibration_Sensor-rescue:main_board_top_rail-ARTS-Lab U5
 U 1 1 629135F7
 P 6650 5400
@@
 	7950 5250 7950 4950
 $Comp
-L ARTS-Lab:power_input U1
+L Vibration_Sensor-rescue:power_input-ARTS-Lab U1
 U 1 1 629E65AA
 P 3050 1600
@@
 $EndComp
 $Comp
-L ARTS-Lab:grounded_DIP_switch switch1
+L Vibration_Sensor-rescue:grounded_DIP_switch-ARTS-Lab switch1
 U 1 1 629E7EFF
 P 4650 950
@@
 	5050 3400 5050 4400
 $Comp
-L ARTS-Lab:nRF24L01+ U6
+L Vibration_Sensor-rescue:nRF24L01+-ARTS-Lab U6
 U 1 1 62C72ED1
 P 7050 3300
@@
 	4650 4600 4300 4600
 Wire Wire Line
-	7900 2950 5050 2950
-Wire Wire Line
 	5050 2950 5050 3400
-Wire Wire Line
-	7900 2950 7900 3000
-Connection ~ 7900 3000
+Connection ~ 5050 3400
 Wire Wire Line
 	7900 3000 7900 3100
-Connection ~ 7900 3100
-Wire Wire Line
-	7900 3100 7900 3200
-Connection ~ 5050 3400
+Wire Wire Line
+	7950 2950 7950 3200
+Wire Wire Line
+	7950 3200 7900 3200
+Wire Wire Line
+	5050 2950 7950 2950
 $EndSCHEMATC
